Commit message: Update README.md Add assets Add top camera Add mission2 assets Implemented draft version of localization but not committed yet

File: src/go1_simulation/urdf/config/sensor.urdf.xacro (robot description, xacro)
@@ -7,5 +7,7 @@
     <xacro:property name="image_format" value="R8G8B8"/>
     <xacro:property name="clip_near" value="0.05"/>
-    <xacro:property name="clip_far" value="3.0"/>
+    <xacro:property name="clip_far" value="100.0"/>
+    <xacro:property name="depth_clip_near" value="0.05"/>
+    <xacro:property name="depth_clip_far" value="7.0"/>
     <xacro:property name="camera_always_on" value="1"/>
     <xacro:property name="camera_update_rate" value="10"/>

File: src/go1_simulation/urdf/robots/go1.urdf.xacro (robot description, xacro)
@@ -8,4 +8,5 @@
     <xacro:include filename="$(find go1_simulation)/urdf/mech/leg.urdf.xacro"/>
     <xacro:include filename="$(find go1_simulation)/urdf/sensors/depthCamera.urdf.xacro"/>
+    <xacro:include filename="$(find go1_simulation)/urdf/mech/cylinder.urdf.xacro"/>
     <xacro:include filename="$(find go1_simulation)/urdf/sensors/imu.urdf.xacro"/>
     <xacro:include filename="$(find go1_simulation)/urdf/sensors/lidar.urdf.xacro"/>
@@ -35,4 +36,8 @@
         <origin rpy="${PI} 0 0" xyz="0.2785 0.0125 0.0167"/>
     </xacro:depthCamera>
+    <xacro:cylinder name='top_camera_cylinder' base_link="trunk" z_offset="0.35" radius="0.01" length="0.30"/>
+    <xacro:depthCamera camID="2" name="top" base_link="top_camera_cylinder">
+        <origin rpy="${PI} 0 0" xyz="0 0 0"/>
+    </xacro:depthCamera>
     <xacro:macro name="material_visual" params="reference ambient diffuse specular">
         <gazebo reference="${reference}">

File: src/go1_simulation/urdf/sensors/depthCamera.urdf.xacro (robot description, xacro)
@@ -1,8 +1,8 @@
 <?xml version="1.0"?>
 <robot xmlns:xacro="http://www.ros.org/wiki/xacro">
-    <xacro:macro name="depthCamera" params="camID name *origin">
+    <xacro:macro name="depthCamera" params="camID name base_link='trunk' *origin">
         <joint name="camera_joint_${name}" type="fixed">
             <xacro:insert_block name="origin"/>
-            <parent link="trunk"/>
+            <parent link="${base_link}"/>
             <child link="camera_${name}"/>
         </joint>
@@ -46,4 +46,10 @@
                         <far>${clip_far}</far>
                     </clip>
+                    <depth_camera>
+                        <clip>
+                            <near>${depth_clip_near}</near>
+                            <far>${depth_clip_far}</far>
+                        </clip>
+                    </depth_camera>
                 </camera>
                 <always_on>${camera_always_on}</always_on>
